Commit message: delet diff_control and fixed the issue missing include velocity_control_plugin.urdf.xacro

File: ugv_ddsm_description/urdf/control/ugv_ddsm_ros2_control.urdf.xacro (robot description, xacro)
@@ -7,37 +7,41 @@
                     <plugin>gz_ros2_control/GazeboSimSystem</plugin>
                 </xacro:if>
+                <xacro:unless value="${use_gazebo}">
+                    <plugin>mock_components/GenericSystem</plugin>
+                    <param name="calculate_dynamics">true</param>
+                </xacro:unless>
             </hardware>
             <joint name="${prefix}front_left_wheel_joint">
               <command_interface name="velocity">
-                  <param name="min">-50.0</param>
-                  <param name="max">50.0</param>
+                  <param name="min">-1.0</param>
+                  <param name="max">1.0</param>
               </command_interface>
               <state_interface name="position"/>
               <state_interface name="velocity"/>
-          </joint>
-          <joint name="${prefix}front_right_wheel_joint">
-              <command_interface name="velocity">
-                  <param name="min">-50.0</param>
-                  <param name="max">50.0</param>
-              </command_interface>
-              <state_interface name="position"/>
-              <state_interface name="velocity"/>
-          </joint>
-          <joint name="${prefix}rear_left_wheel_joint">
-              <command_interface name="velocity">
-                  <param name="min">-50.0</param>
-                  <param name="max">50.0</param>
-              </command_interface>
-              <state_interface name="position"/>
-              <state_interface name="velocity"/>
-          </joint>
-          <joint name="${prefix}rear_right_wheel_joint">
-              <command_interface name="velocity">
-                  <param name="min">-50.0</param>
-                  <param name="max">50.0</param>
-              </command_interface>
-              <state_interface name="position"/>
-              <state_interface name="velocity"/>
-          </joint>
+            </joint>
+            <joint name="${prefix}front_right_wheel_joint">
+                <command_interface name="velocity">
+                    <param name="min">-1.0</param>
+                    <param name="max">1.0</param>
+                </command_interface>
+                <state_interface name="position"/>
+                <state_interface name="velocity"/>
+            </joint>
+            <joint name="${prefix}rear_left_wheel_joint">
+                <command_interface name="velocity">
+                    <param name="min">-1.0</param>
+                    <param name="max">1.0</param>
+                </command_interface>
+                <state_interface name="position"/>
+                <state_interface name="velocity"/>
+            </joint>
+            <joint name="${prefix}rear_right_wheel_joint">
+                <command_interface name="velocity">
+                    <param name="min">-1.0</param>
+                    <param name="max">1.0</param>
+                </command_interface>
+                <state_interface name="position"/>
+                <state_interface name="velocity"/>
+            </joint>
       </ros2_control>
   </xacro:macro>

File: ugv_ddsm_description/urdf/control/velocity_control_plugin.urdf.xacro (robot description, xacro)
@@ -13,4 +13,7 @@
             </gazebo>
         </xacro:if>
+    <xacro:unless value="$(arg use_gazebo)">
+        <!-- todo: -->
+    </xacro:unless>
     </xacro:macro>
 </robot>

File: ugv_ddsm_description/urdf/robots/Robot_wrapper.urdf.xacro (robot description, xacro)
@@ -6,4 +6,6 @@
     <xacro:include filename="$(find ugv_ddsm_description)/urdf/mech/Robot.urdf"/>
     <xacro:include filename="$(find ugv_ddsm_description)/urdf/mech/Robot_sensors.urdf.xacro"/>
+    <xacro:include filename="$(find ugv_ddsm_description)/urdf/control/velocity_control_plugin.urdf.xacro" />
+    <xacro:load_velocity_control_plugin use_gazebo="$(arg use_gazebo)"/>
     <xacro:include filename="$(find ugv_ddsm_description)/urdf/control/gazebo_sim_ros2_control.urdf.xacro" />
     <xacro:load_gazebo_sim_ros2_control_plugin
